File: hardware/SensorHub.kicad_pcb (KiCad board)
At the start: 2 copper layers, 72 x 50 mm, 43 parts, among them IC1 VEML6070, IC2 LT3652EMSE, IC3 BME680, IC4 BH1726, IC5 MCP9808, M1 ParticleArgon, SW1 ENABLE, X1 WIND, X2 SOLAR

Commit message: Clean up hardware files
Parts:
- removed C1: 1uF, Capacitor_SMD:C_0805_2012Metric_Pad1.15x1.40mm_HandSolder
- R8: value NB -> 100k
- R9: value NB -> 22k
- moved C9 0.52 mm to (180.2, 116.3)
Connections:
- IC2 pad 6: Net-(C1-Pad2) -> GND
Routing:
- net GND: track 27.4 -> 29.8 mm
- net Net-(C1-Pad2): track 1.64 -> 0.00 mm

Commit message: Optimize LTC3652 layout
Parts:
- moved C4 10.2 mm to (176.3, 101.1), turned to 180 degrees
- moved C5 5.41 mm to (180.5, 101.1)
- moved R2 4.35 mm to (161.0, 96.3), turned to 180 degrees
- moved R15 3.84 mm to (153.9, 95.5)
- moved R9 2.02 mm to (179.5, 119.1)
- moved C9 1.70 mm to (178.6, 117.1)
- moved R8 0.63 mm to (175.6, 119.1)
- moved D2 0.13 mm to (176.2, 104.0)
- moved M1 0.13 mm to (168.8, 88.5)
- moved D1 0.09 mm to (168.2, 108.2)
Routing:
- net Net-(M1-Pad5): track 46.1 -> 58.4 mm, vias 0 -> 1
- net /~CHRG: track 49.8 -> 40.5 mm, vias 1 -> 3
- net GND: track 29.8 -> 34.0 mm
- net Net-(IC2-Pad2): track 12.0 -> 13.4 mm
- net /~FAULT: track 41.7 -> 40.7 mm, vias 1 -> 3
- net /~TempAlert: track 23.5 -> 22.7 mm
- net Net-(M1-Pad27): track 40.2 -> 40.9 mm
- net /WindSensor: track 38.5 -> 38.7 mm, vias 0 -> 1
Other:
- board text added: "1.2"
- board text removed: "1.1"
